File: jackco-esp32-pico/jackco-esp32-pico-panel-v2.kicad_pcb (KiCad board)
At the start: 2 copper layers, 105 x 105 mm, 116 parts, among them J1 USB, J2 GPIO, J3 GPIO, J4 VUSB, Q1 S8050, Q2 S8050, SW1 BOOT, SW2 RESET, U1 ESP32-PICO-D4, U2 ESP-PSRAM32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

Commit message: Move panelized board Vcut to outline layer
Parts:
- added REF**: NPTH, NPTH, F.Cu at (34.1, 146.2)
- added REF**: NPTH, NPTH, F.Cu at (123.1, 52.2)
- added REF**: NPTH, NPTH, F.Cu at (34.1, 52.2)
- added REF**: Fiducial, Fiducial, B.Cu at (39.1, 146.2)
- added REF**: Fiducial, Fiducial, F.Cu at (39.1, 146.2)
- added REF**: Fiducial, Fiducial, B.Cu at (118.1, 52.2)
- added REF**: Fiducial, Fiducial, F.Cu at (118.1, 52.2)
- added REF**: Fiducial, Fiducial, B.Cu at (39.1, 52.2)
- added REF**: Fiducial, Fiducial, F.Cu at (39.1, 52.2)
Changed lines of the file:
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@@
   (general
     (thickness 1.6)
-    (drawings 158)
+    (drawings 174)
     (tracks 2080)
     (zones 0)
-    (modules 116)
+    (modules 125)
     (nets 257)
   )
@@
       (outputformat 1)
       (mirror false)
-      (drillshape 0)
+      (drillshape 1)
       (scaleselection 1)
-      (outputdirectory "gerber"))
+      (outputdirectory ""))
   )
   (net 0 "")
@@
     (add_net Board_4-VDD_SDIO)
   )
+  (module NPTH (layer F.Cu)
+    (at 34.075003 146.21201)
+    (fp_text reference REF** (at 0 0.5) (layer F.SilkS) hide
+      (effects (font (size 1 1) (thickness 0.15)))
+    )
+    (fp_text value NPTH (at 0 -0.5) (layer F.Fab) hide
+      (effects (font (size 1 1) (thickness 0.15)))
+    )
+    (pad "" np_thru_hole circle (at 0 0) (size 1.5 1.5) (drill 1.5) (layers *.Cu *.Mask))
+  )
+  (module NPTH (layer F.Cu)
+    (at 123.075002 52.21201)
+    (fp_text reference REF** (at 0 0.5) (layer F.SilkS) hide
+      (effects (font (size 1 1) (thickness 0.15)))
+    )
+    (fp_text value NPTH (at 0 -0.5) (layer F.Fab) hide
+      (effects (font (size 1 1) (thickness 0.15)))
+    )
+    (pad "" np_thru_hole circle (at 0 0) (size 1.5 1.5) (drill 1.5) (layers *.Cu *.Mask))
+  )
+  (module NPTH (layer F.Cu)
+    (at 34.075003 52.21201)
+    (fp_text reference REF** (at 0 0.5) (layer F.SilkS) hide
+      (effects (font (size 1 1) (thickness 0.15)))
+    )
+    (fp_text value NPTH (at 0 -0.5) (layer F.Fab) hide
+      (effects (font (size 1 1) (thickness 0.15)))
+    )
+    (pad "" np_thru_hole circle (at 0 0) (size 1.5 1.5) (drill 1.5) (layers *.Cu *.Mask))
+  )
+  (module Fiducial (layer B.Cu)
+    (at 39.075003 146.21201)
+    (descr "Circular Fiducial")
+    (tags fiducial)
+    (attr smd)
+    (fp_text reference REF** (at 0 1.5) (layer B.SilkS) hide
+      (effects (font (size 1 1) (thickness 0.15)) (justify mirror))
+    )
+    (fp_text value Fiducial (at 0 -1.5) (layer B.Fab) hide
+      (effects (font (size 1 1) (thickness 0.15)) (justify mirror))
+    )
+    (pad "" smd circle (at 0 0) (size 1 1) (layers B.Cu B.Mask)
+      (solder_mask_margin 0.5) (clearance 0.5))
+  )
+  (module Fiducial (layer F.Cu)
+    (at 39.075003 146.21201)
+    (descr "Circular Fiducial")
+    (tags fiducial)
+    (attr smd)
+    (fp_text reference REF** (at 0 -1.5) (layer F.SilkS) hide
+      (effects (font (size 1 1) (thickness 0.15)))
+    )
+    (fp_text value Fiducial (at 0 1.5) (layer F.Fab) hide
+      (effects (font (size 1 1) (thickness 0.15)))
+    )
+    (pad "" smd circle (at 0 0) (size 1 1) (layers F.Cu F.Mask)
+      (solder_mask_margin 0.5) (clearance 0.5))
+  )
+  (module Fiducial (layer B.Cu)
+    (at 118.075002 52.21201)
+    (descr "Circular Fiducial")
+    (tags fiducial)
+    (attr smd)
+    (fp_text reference REF** (at 0 1.5) (layer B.SilkS) hide
+      (effects (font (size 1 1) (thickness 0.15)) (justify mirror))
+    )
+    (fp_text value Fiducial (at 0 -1.5) (layer B.Fab) hide
+      (effects (font (size 1 1) (thickness 0.15)) (justify mirror))
+    )
+    (pad "" smd circle (at 0 0) (size 1 1) (layers B.Cu B.Mask)
+      (solder_mask_margin 0.5) (clearance 0.5))
+  )
+  (module Fiducial (layer F.Cu)
+    (at 118.075002 52.21201)
+    (descr "Circular Fiducial")
+    (tags fiducial)
+    (attr smd)
+    (fp_text reference REF** (at 0 -1.5) (layer F.SilkS) hide
+      (effects (font (size 1 1) (thickness 0.15)))
+    )
+    (fp_text value Fiducial (at 0 1.5) (layer F.Fab) hide
+      (effects (font (size 1 1) (thickness 0.15)))
+    )
+    (pad "" smd circle (at 0 0) (size 1 1) (layers F.Cu F.Mask)
+      (solder_mask_margin 0.5) (clearance 0.5))
+  )
+  (module Fiducial (layer B.Cu)
+    (at 39.075003 52.21201)
+    (descr "Circular Fiducial")
+    (tags fiducial)
+    (attr smd)
+    (fp_text reference REF** (at 0 1.5) (layer B.SilkS) hide
+      (effects (font (size 1 1) (thickness 0.15)) (justify mirror))
+    )
+    (fp_text value Fiducial (at 0 -1.5) (layer B.Fab) hide
+      (effects (font (size 1 1) (thickness 0.15)) (justify mirror))
+    )
+    (pad "" smd circle (at 0 0) (size 1 1) (layers B.Cu B.Mask)
+      (solder_mask_margin 0.5) (clearance 0.5))
+  )
+  (module Fiducial (layer F.Cu)
+    (at 39.075003 52.21201)
+    (descr "Circular Fiducial")
+    (tags fiducial)
+    (attr smd)
+    (fp_text reference REF** (at 0 -1.5) (layer F.SilkS) hide
+      (effects (font (size 1 1) (thickness 0.15)))
+    )
+    (fp_text value Fiducial (at 0 1.5) (layer F.Fab) hide
+      (effects (font (size 1 1) (thickness 0.15)))
+    )
+    (pad "" smd circle (at 0 0) (size 1 1) (layers F.Cu F.Mask)
+      (solder_mask_margin 0.5) (clearance 0.5))
+  )
   (module AN9520:SMD_ANT9520 (layer F.Cu)
     (at 51.778001 132.692016 90)
@@
   )
   (gr_line (start 26.075003 123.82) (end 131.075002 123.82) (layer Edge.Cuts) (width 0.4))
-  (gr_line (start 29.075 148.712) (end 29.075 49.712) (layer Edge.Cuts) (width 0.1))
-  (gr_line (start 128.075 148.712) (end 29.075 148.712) (layer Edge.Cuts) (width 0.1))
-  (gr_line (start 128.075 49.712) (end 128.075 148.712) (layer Edge.Cuts) (width 0.1))
-  (gr_line (start 29.075 49.712) (end 128.075 49.712) (layer Edge.Cuts) (width 0.1))
+  (gr_line (start 29.0758 49.7212) (end 29.075 49.7361) (layer Edge.Cuts) (width 0.1))
+  (gr_line (start 29.079 49.7153) (end 29.0758 49.7212) (layer Edge.Cuts) (width 0.1))
+  (gr_line (start 29.0842 49.7128) (end 29.079 49.7153) (layer Edge.Cuts) (width 0.1))
+  (gr_line (start 29.0996 49.712) (end 29.0842 49.7128) (layer Edge.Cuts) (width 0.1))
+  (gr_line (start 128.0505 49.712) (end 29.0996 49.712) (layer Edge.Cuts) (width 0.1))
+  (gr_line (start 128.0658 49.7128) (end 128.0505 49.712) (layer Edge.Cuts) (width 0.1))
+  (gr_line (start 128.071 49.7153) (end 128.0658 49.7128) (layer Edge.Cuts) (width 0.1))
+  (gr_line (start 128.0742 49.7212) (end 128.071 49.7153) (layer Edge.Cuts) (width 0.1))
+  (gr_line (start 128.075 49.7366) (end 128.0742 49.7212) (layer Edge.Cuts) (width 0.1))
+  (gr_line (start 128.075 148.6875) (end 128.075 49.7366) (layer Edge.Cuts) (width 0.1))
+  (gr_line (start 128.0742 148.7028) (end 128.075 148.6875) (layer Edge.Cuts) (width 0.1))
+  (gr_line (start 128.0717 148.708) (end 128.0742 148.7028) (layer Edge.Cuts) (width 0.1))
+  (gr_line (start 128.0658 148.7112) (end 128.0717 148.708) (layer Edge.Cuts) (width 0.1))
+  (gr_line (start 128.0505 148.712) (end 128.0658 148.7112) (layer Edge.Cuts) (width 0.1))
+  (gr_line (start 29.0996 148.712) (end 128.0505 148.712) (layer Edge.Cuts) (width 0.1))
+  (gr_line (start 29.0842 148.7112) (end 29.0996 148.712) (layer Edge.Cuts) (width 0.1))
+  (gr_line (start 29.079 148.7087) (end 29.0842 148.7112) (layer Edge.Cuts) (width 0.1))
+  (gr_line (start 29.0758 148.7028) (end 29.079 148.7087) (layer Edge.Cuts) (width 0.1))
+  (gr_line (start 29.075 148.6875) (end 29.0758 148.7028) (layer Edge.Cuts) (width 0.1))
+  (gr_line (start 29.075 49.7361) (end 29.075 148.6875) (layer Edge.Cuts) (width 0.1))
   (gr_text 3v3 (at 54.624001 142.376016 90) (layer F.SilkS)
     (effects (font (size 1 1) (thickness 0.15)))
