File: jackco-esp32-pico/jackco-esp32-pico-panel-v2.kicad_pcb (KiCad board)
At the start: 2 copper layers, 105 x 105 mm, 116 parts, among them J1 USB, J2 GPIO, J3 GPIO, J4 VUSB, Q1 S8050, Q2 S8050, SW1 BOOT, SW2 RESET, U1 ESP32-PICO-D4, U2 ESP-PSRAM32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

Commit message: Final adjustments for Rev 2.1
Parts:
- removed the R4 at (102.6, 132.9)
- removed the R4 at (102.6, 108.3)
- removed the R4 at (102.6, 83.7)
- removed the R4 at (102.6, 59.1)
- removed the R5 at (102.6, 135.8)
- removed the R5 at (102.6, 111.2)
- removed the R5 at (102.6, 86.6)
- removed the R5 at (102.6, 62.0)
- added R4: 5.11K, Resistor_SMD:R_0603_1608Metric_Pad1.05x0.95mm_HandSolder, F.Cu at (103.8, 132.8)
- added R4: 5.11K, Resistor_SMD:R_0603_1608Metric_Pad1.05x0.95mm_HandSolder, F.Cu at (103.8, 108.2)
- added R4: 5.11K, Resistor_SMD:R_0603_1608Metric_Pad1.05x0.95mm_HandSolder, F.Cu at (103.8, 83.6)
- added R4: 5.11K, Resistor_SMD:R_0603_1608Metric_Pad1.05x0.95mm_HandSolder, F.Cu at (103.8, 59.0)
- added R5: 5.11K, Resistor_SMD:R_0603_1608Metric_Pad1.05x0.95mm_HandSolder, F.Cu at (103.7, 135.7)
- added R5: 5.11K, Resistor_SMD:R_0603_1608Metric_Pad1.05x0.95mm_HandSolder, F.Cu at (103.7, 111.1)
- added R5: 5.11K, Resistor_SMD:R_0603_1608Metric_Pad1.05x0.95mm_HandSolder, F.Cu at (103.7, 86.5)
- added R5: 5.11K, Resistor_SMD:R_0603_1608Metric_Pad1.05x0.95mm_HandSolder, F.Cu at (103.7, 61.9)
- added REF**: NPTH, NPTH, F.Cu at (31.6, 145.7)
- added REF**: NPTH, NPTH, F.Cu at (125.6, 52.7)
- added REF**: NPTH, NPTH, F.Cu at (31.6, 52.7)
- added REF**: Fiducial, Fiducial, B.Cu at (31.6, 142.7)
- added REF**: Fiducial, Fiducial, F.Cu at (31.6, 142.7)
- added REF**: Fiducial, Fiducial, B.Cu at (125.6, 55.7)
- added REF**: Fiducial, Fiducial, F.Cu at (125.6, 55.7)
- added REF**: Fiducial, Fiducial, B.Cu at (31.6, 55.7)
- added REF**: Fiducial, Fiducial, F.Cu at (31.6, 55.7)
- R6 (x4): value 330 -> 470
Routing:
- net Board_4-GND: track 70.8 -> 62.7 mm, vias 100 -> 107
- net Board_1-GND: track 70.8 -> 62.7 mm, vias 100 -> 107
- net Board_3-GND: track 70.8 -> 62.7 mm, vias 100 -> 107
- net Board_2-GND: track 70.8 -> 62.7 mm, vias 100 -> 107
- net Board_4-+5V: track 48.1 -> 44.9 mm, vias 2 -> 3
- net Board_2-+5V: track 48.1 -> 44.9 mm, vias 2 -> 3
- net Board_1-+5V: track 48.1 -> 44.9 mm, vias 2 -> 3
- net Board_3-+5V: track 48.1 -> 44.9 mm, vias 2 -> 3
- net Board_2-Net-(J1-PadA5): track 4.73 -> 3.69 mm
- net Board_3-Net-(J1-PadA5): track 4.73 -> 3.69 mm
- net Board_1-Net-(J1-PadA5): track 4.73 -> 3.69 mm
- net Board_4-Net-(J1-PadA5): track 4.73 -> 3.69 mm
Other:
- board text added: "IO15"
- board text added: "Rev. 2.1"
- board text removed: "Rev. 2"

Commit message: Final adjustments for Rev 2.1
Parts:
- removed the Q2 at (84.6, 141.5)
- removed the Q2 at (84.6, 92.3)
- removed the REF** at (31.6, 142.7) (x2)
- removed the REF** at (125.6, 55.7) (x2)
- removed the REF** at (31.6, 55.7) (x2)
- removed the U4 at (86.5, 133.9)
- added J1: USB, Connector_USB:USB_C_Receptacle_HRO_TYPE-C-31-M-12, B.Cu at (103.3, 134.1)
- added R1: 10K, Resistor_SMD:R_0603_1608Metric_Pad1.05x0.95mm_HandSolder, B.Cu at (69.6, 93.1)
- added R2: 10K, Resistor_SMD:R_0603_1608Metric_Pad1.05x0.95mm_HandSolder, B.Cu at (88.1, 142.4)
- added REF**: Fiducial, Fiducial, B.Cu at (31.6, 142.7)
- added REF**: Fiducial, Fiducial, F.Cu at (31.6, 142.7)
- added REF**: Fiducial, Fiducial, B.Cu at (125.6, 55.7)
- added REF**: Fiducial, Fiducial, F.Cu at (125.6, 55.7)
- added REF**: Fiducial, Fiducial, B.Cu at (31.6, 55.7)
- added REF**: Fiducial, Fiducial, F.Cu at (31.6, 55.7)
- Q2: renamed from R2; value 10K -> S8050; footprint Resistor_SMD:R_0603_1608Metric_Pad1.05x0.95mm_HandSolder -> Package_TO_SOT_SMD:SOT-23
- Q2: renamed from R1; value 10K -> S8050; footprint Resistor_SMD:R_0603_1608Metric_Pad1.05x0.95mm_HandSolder -> Package_TO_SOT_SMD:SOT-23
- U4: renamed from J1; value USB -> AMS1117; footprint Connector_USB:USB_C_Receptacle_HRO_TYPE-C-31-M-12 -> Package_TO_SOT_SMD:SOT-223-3_TabPin2
- moved U4 16.8 mm to (86.5, 133.9), turned to 0 degrees
- moved Q2 15.0 mm to (84.6, 92.3), turned to 180 degrees
- moved Q2 3.60 mm to (84.6, 141.5)
Connections:
- Q2 pad 1: Board_4-Net-(Q1-Pad1) -> Board_4-Net-(Q2-Pad1)
- Q2 pad 1: Board_2-3v3A -> Board_2-Net-(Q2-Pad1)
- Q2 pad 2: Board_2-EN -> Board_2-RTS
Routing:
- net Board_2-SENSE_CAPN: track 8.81 -> 7.85 mm
- net Board_3-SENSE_CAPN: track 8.81 -> 7.85 mm
- net Board_4-SENSE_CAPN: track 8.81 -> 7.85 mm
- net Board_1-SENSE_CAPN: track 8.81 -> 7.85 mm
- net Board_3-SENSE_VN: track 10.2 -> 9.37 mm
- net Board_1-SENSE_VN: track 10.2 -> 9.37 mm
- net Board_2-SENSE_VN: track 10.2 -> 9.37 mm
- net Board_4-SENSE_VN: track 10.2 -> 9.37 mm
- net Board_4-GND: vias 107 -> 104
- net Board_3-GND: vias 107 -> 104
- net Board_2-GND: vias 107 -> 104
- net Board_1-GND: vias 107 -> 104
Other:
- board size 105 x 105 mm -> 99 x 99 mm
