File: jackco-esp32-pico/jackco-esp32-pico-panel-v2.kicad_pcb (KiCad board)
At the start: 2 copper layers, 99 x 99 mm, 125 parts, among them J1 USB, J2 GPIO, J3 GPIO, J4 VUSB, Q1 S8050, Q2 S8050, SW1 BOOT, SW2 RESET, U1 ESP32-PICO-D4, U2 ESP-PSRAM32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

Commit message: Generate gerber for Rev 2.1
Other:
- board size 99 x 99 mm -> 105 x 105 mm
