File: jackco-esp32-pico/jackco-esp32-pico.sch (KiCad schematic (older format))
At the start: 29 parts, among them J1 USB, J2 GPIO, J3 GPIO, J4 VUSB, Q1 S8050, Q2 S8050, SW1 BOOT, SW2 RESET, U1 ESP32-PICO-D4, U2 ESP-PSRAM32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

Commit message: Add PDFs, rename project
Other:
- note added: "1"
- note added: "8 Aug 2020"
- note added: "JackcoESP32-PICO Rev 1"
- note removed: "Borscht-ESP32-Pico"
Changed lines of the file:
@@
 Connection ~ 6500 6750
 Text Notes 7400 7500 0    50   ~ 0
-Borscht-ESP32-Pico
+JackcoESP32-PICO Rev 1
 $Comp
 L Device:R_Small R6
@@
 Wire Wire Line
 	4550 6500 4550 6650
+Text Notes 10600 7650 0    50   ~ 0
+1
+Text Notes 8150 7650 0    50   ~ 0
+8 Aug 2020
 $EndSCHEMATC

Commit message: Redesign 5v domain, fix wrong S8050
Parts:
- ANT1: symbol AN9520:AN9520 -> jackco-esp32-pico-rescue:AN9520-AN9520
- J1: symbol Connector:USB_C_Receptacle_USB2.0 -> jackco-esp32-pico-rescue:USB_C_Receptacle_USB2.0-Connector
- Q1, Q2: symbol Transistor_BJT:S8050 -> dk_Transistors-Bipolar-BJT-Single:MMSS8050-H-TP
Connections:
- net DTR: now also Q1.2 (E); no longer Q1.1 (E)
- net RTS: now also Q2.2 (E); no longer Q2.1 (E)
- net at R3.1: now also Q2.1 (B); no longer Q2.2 (B)
- net at R2.1: now also Q1.1 (B); no longer Q1.2 (B)
Changed lines of the file:
@@
 Connection ~ 7300 2200
-$Comp
-L power:+3.3V #PWR0105
-U 1 1 5F2E8E41
-P 4700 800
-F 0 "#PWR0105" H 4700 650 50  0001 C CNN
-F 1 "+3.3V" H 4715 973 50  0000 C CNN
-F 2 "" H 4700 800 50  0001 C CNN
-F 3 "" H 4700 800 50  0001 C CNN
-	1    4700 800
-	1    0    0    -1
-$EndComp
 $Comp
 L Device:R_Small R1
@@
 Connection ~ 800  2950
 $Comp
-L Transistor_BJT:S8050 Q2
+L dk_Transistors-Bipolar-BJT-Single:MMSS8050-H-TP Q2
 U 1 1 5F35268D
 P 1650 1200
@@
 RTS
 $Comp
-L Transistor_BJT:S8050 Q1
+L dk_Transistors-Bipolar-BJT-Single:MMSS8050-H-TP Q1
 U 1 1 5F35441F
 P 3600 1200
@@
 	1100 1200 950  1200
 $Comp
-L Connector:USB_C_Receptacle_USB2.0 J1
+L jackco-esp32-pico-rescue:USB_C_Receptacle_USB2.0-Connector J1
 U 1 1 5F3A031B
 P 1050 6300
@@
 NoConn ~ 8200 3350
 $Comp
-L AN9520:AN9520 ANT1
+L jackco-esp32-pico-rescue:AN9520-AN9520 ANT1
 U 1 1 5F783087
 P 8900 2650
@@
 Text Notes 8150 7650 0    50   ~ 0
 8 Aug 2020
+Text GLabel 7750 1800 2    50   Input ~ 0
+3v3A
+Wire Wire Line
+	7500 1800 7750 1800
+Text GLabel 4700 800  1    50   Input ~ 0
+3v3A
 $EndSCHEMATC

Commit message: Final adjustments for Rev 2.1
Parts:
- R6: value 330 -> 470
Changed lines of the file:
@@
 P 4850 3450
 F 0 "R6" H 4909 3496 50  0000 L CNN
-F 1 "330" H 4909 3405 50  0000 L CNN
+F 1 "470" H 4909 3405 50  0000 L CNN
 F 2 "Resistor_SMD:R_0603_1608Metric_Pad1.05x0.95mm_HandSolder" H 4850 3450 50  0001 C CNN
 F 3 "~" H 4850 3450 50  0001 C CNN
