File: jackco-esp32-pico/jackco-esp32-pico.kicad_pcb (KiCad board)
At the start: 2 copper layers, 57.2 x 24.6 mm, 29 parts, among them J1 USB, J2 GPIO, J3 GPIO, J4 VUSB, Q1 S8050, Q2 S8050, SW1 BOOT, SW2 RESET, U1 ESP32-PICO-D4, U2 ESP-PSRAM32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

Commit message: Redesign 5v domain, fix wrong S8050
Parts:
- C9, R1: moved to B.Cu
- moved R1 27.2 mm to (105.7, 122.4), turned to 270 degrees
- moved SW2 21.7 mm to (114.0, 121.9), turned to 180 degrees
- moved C2 21.4 mm to (107.7, 122.5), turned to 90 degrees
- moved SW1 20.9 mm to (134.6, 121.4), turned to 0 degrees
- moved C9 18.8 mm to (113.6, 119.5)
- moved Q2 7.44 mm to (120.7, 121.6), turned to 180 degrees
- moved Q1 6.87 mm to (127.7, 121.5), turned to 0 degrees
- moved R3 2.20 mm to (124.2, 120.5), turned to 0 degrees
- moved R2 1.83 mm to (124.2, 122.5), turned to 180 degrees
- moved C6 1.42 mm to (123.1, 107.7)
- moved C3 0.69 mm to (115.9, 116.6)
- moved U2 0.06 mm to (109.7, 114.7)
Connections:
- net +3V3 renamed 3v3A
- ANT1 pad P$GND: Net-(ANT1-PadP$GND) -> (no net)
- J1 pad A8: Net-(J1-PadA8) -> (no net)
- J1 pad B8: Net-(J1-PadB8) -> (no net)
- Q1 pad 1: DTR -> Net-(Q1-Pad1)
- Q1 pad 2: Net-(Q1-Pad2) -> DTR
- Q2 pad 1: RTS -> Net-(Q2-Pad1)
- Q2 pad 2: Net-(Q2-Pad2) -> RTS
- R2 pad 1: Net-(Q1-Pad2) -> Net-(Q1-Pad1)
- R3 pad 1: Net-(Q2-Pad2) -> Net-(Q2-Pad1)
- U1 pad 10: Net-(U1-Pad10) -> (no net)
- U1 pad 11: Net-(U1-Pad11) -> (no net)
- U1 pad 25: Net-(U1-Pad25) -> (no net)
- U1 pad 28: Net-(U1-Pad28) -> (no net)
- U1 pad 44: Net-(U1-Pad44) -> (no net)
- U1 pad 45: Net-(U1-Pad45) -> (no net)
- U1 pad 47: Net-(U1-Pad47) -> (no net)
- U1 pad 48: Net-(U1-Pad48) -> (no net)
- U3 pad 10: Net-(U3-Pad10) -> (no net)
- U3 pad 11: Net-(U3-Pad11) -> (no net)
- U3 pad 12: Net-(U3-Pad12) -> (no net)
- U3 pad 15: Net-(U3-Pad15) -> (no net)
- U3 pad 7: Net-(U3-Pad7) -> (no net)
- U3 pad 8: Net-(U3-Pad8) -> (no net)
- U3 pad 9: Net-(U3-Pad9) -> (no net)
Routing:
- net GND: track 138.0 -> 70.8 mm, vias 51 -> 100
- net EN: track 50.2 -> 28.6 mm, vias 2 -> 1
- net IO0: track 49.0 -> 38.8 mm
- net Net-(Q2-Pad2): track 4.53 -> 0.00 mm
- net DTR: track 11.6 -> 8.23 mm
- net 3v3A: track 99.3 -> 102.2 mm, vias 6 -> 4
- net +5V: track 46.0 -> 48.1 mm, vias 3 -> 2
- net Net-(Q1-Pad2): track 1.89 -> 0.00 mm
- net Net-(Q2-Pad1): track 0.00 -> 1.71 mm
- net Net-(Q1-Pad1): track 0.00 -> 1.64 mm
- net RTS: track 6.98 -> 8.53 mm
- net IO32: track 8.65 -> 9.20 mm
Other:
- board text added: "Rev. 2"
- board text removed: "IO15"
- board text removed: "Rev. 1"

Commit message: Final adjustments for Rev 2.1
Parts:
- R6: value 330 -> 470
- moved R4 1.22 mm to (139.9, 112.9)
- moved R5 1.19 mm to (139.8, 115.8)
Routing:
- net GND: track 70.8 -> 62.7 mm, vias 100 -> 107
- net +5V: track 48.1 -> 44.9 mm, vias 2 -> 3
- net Net-(J1-PadA5): track 4.73 -> 3.69 mm
Other:
- board text added: "IO15"
- board text added: "Rev. 2.1"
- board text removed: "Rev. 2"

Commit message: Final adjustments for Rev 2.1
Routing:
- net SENSE_CAPN: track 8.81 -> 7.85 mm
- net SENSE_VN: track 10.2 -> 9.37 mm
- net GND: vias 107 -> 104
